File: ILI9341_ESP32_V1/ILI9341_ESP32_V1.kicad_pcb (KiCad board)
At the start: 2 copper layers, 81 x 113 mm, 72 parts, among them J1 USB_C_Receptacle_USB2.0_16P, J2 Conn_01x02_Female, J3 Conn_01x02_Female, J4 Conn_01x18_Socket, Q1 BC807, SW1 SW_DIP_x01, SW10 SW_Push, SW11 SW_Push, SW12 SW_Push, SW13 SW_Wuerth_450301014042, SW2 SW_Push, SW3 SW_Push, SW4 SW_Push, SW5 SW_Push, SW6 SW_Push, SW7 SW_Push, SW8 SW_Push, SW9 SW_Push, U1 MCP73831-2-OT, U2 XM5062S, U3 ESP32-S3-WROOM-2, U4 3_2_ZOLL_ILI9341, U5 MAX98357AETE+T, U6 02FVS3, U7 02FVS3

Commit message: Add new connection (inter PCB)
build up new concept to fit in original gameboy case :) hope so
sound tested on prototyp wirering
Parts:
- removed R24: 22, Resistor_SMD:R_0603_1608Metric_Pad0.98x0.95mm_HandSolder
- added C8: 4µ7, Capacitor_SMD:C_1206_3216Metric, F.Cu at (159.9, 83.5)
- added C9: 4µ7, Capacitor_SMD:C_1206_3216Metric, B.Cu at (110.2, 85.2)
- added J5: Micro_SD_Card_CD, TheBrutzlers_Lib:MicroSD_Self_ bomb, B.Cu at (105.1, 75.2)
- added J7: Conn_01x18_Socket, TheBrutzlers_Lib:solder connector 0.8mm 18 pin, F.Cu at (124.0, 74.0)
- added U8: IPCB05501F20S3V, easyeda2kicad:CONN-SMD_20P-P0.50_INCP_IPCB05501F20S3V, F.Cu at (196.1, 142.3)
- added U9: IPCB05501M20S3V, easyeda2kicad:CONN-SMD_20P-P0.50_INCP_IPCB05501M20S3V, B.Cu at (110.2, 107.6)
- J1, U3, U7: moved to F.Cu
- J2, J3, R6, R7, SW6, SW8: moved to B.Cu
- R23: value 22 -> 10
- moved LS1 195.5 mm to (218.7, 27.0)
- moved SW7 189.5 mm to (34.9, 74.1)
- moved J2 161.5 mm to (190.2, 42.2), turned to 180 degrees
- moved SW6 144.4 mm to (81.4, 89.2), turned to 90 degrees
- moved SW8 142.9 mm to (67.6, 98.0), turned to 90 degrees
- moved D2 131.4 mm to (195.6, 24.6)
- moved FB2 125.9 mm to (212.7, 28.8)
- moved D1 125.3 mm to (195.6, 28.2)
- moved FB1 125.2 mm to (212.7, 26.8)
- moved R3 123.9 mm to (116.0, 65.5), turned to 180 degrees
- moved U5 122.8 mm to (207.8, 26.0)
- moved R19 122.3 mm to (125.0, 91.5), turned to -90 degrees
- moved R17 121.2 mm to (126.5, 91.5), turned to 90 degrees
- moved R23 120.6 mm to (126.5, 87.5), turned to 90 degrees
- moved R18 119.5 mm to (128.0, 91.5), turned to -90 degrees
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Connections:
- J4 pad 7: unconnected-(J4-Pin_7-Pad7) -> Net-(J4-Pin_7)
- J4 pad 9: unconnected-(J4-Pin_9-Pad9) -> +3V3
- R23 pad 1: Net-(R23-Pad1) -> GND
- R23 pad 2: +3V3 -> Net-(J6-Pin_7)
- SW10 pad 1: Net-(R23-Pad1) -> /FRONT_BUTTONS/GND
- SW10 pad 2: /KEY_SELECT -> /FRONT_BUTTONS/SELECT
- SW11 pad 1: Net-(R23-Pad1) -> /FRONT_BUTTONS/GND
- SW11 pad 2: /KEY_A -> /FRONT_BUTTONS/A
- SW12 pad 1: Net-(R23-Pad1) -> /FRONT_BUTTONS/GND
- SW12 pad 2: /KEY_B -> /FRONT_BUTTONS/B
- SW2 pad 1: +3V3 -> /FRONT_BUTTONS/3V3
- SW2 pad 2: /KEY_RIGHT -> /FRONT_BUTTONS/RIGHT
- SW3 pad 1: +3V3 -> /FRONT_BUTTONS/3V3
- SW3 pad 2: /KEY_LEFT -> /FRONT_BUTTONS/LEFT
- SW4 pad 1: +3V3 -> /FRONT_BUTTONS/3V3
- SW4 pad 2: /KEY_UP -> /FRONT_BUTTONS/UP
- SW5 pad 1: +3V3 -> /FRONT_BUTTONS/3V3
- SW5 pad 2: /KEY_DOWN -> /FRONT_BUTTONS/DOWN
- SW6 pad 1: Net-(R23-Pad1) -> GND
- SW7 pad 1: Net-(R23-Pad1) -> GND
- SW8 pad 1: Net-(R23-Pad1) -> GND
- SW9 pad 1: Net-(R23-Pad1) -> /FRONT_BUTTONS/GND
- SW9 pad 2: /KEY_START -> /FRONT_BUTTONS/START
- U6 pad A: unconnected-(U6-PadA) -> /KEY_OPTION
- U6 pad C: unconnected-(U6-PadC) -> GND
- U6 pad S: unconnected-(U6-PadS) -> /KEY_VOL_BOOT
- U7 pad A: unconnected-(U7-PadA) -> /KEY_OPTION
- U7 pad C: unconnected-(U7-PadC) -> GND
- U7 pad S: unconnected-(U7-PadS) -> /KEY_MENU
Routing:
- net GND: track 0.00 -> 21.8 mm, vias 0 -> 3
- net +3V3: track 0.00 -> 9.91 mm, vias 0 -> 1
- net Net-(U2-FB): track 0.00 -> 6.02 mm
- net Net-(U1-PROG): track 0.00 -> 4.21 mm
- net /VUSB: track 0.00 -> 4.19 mm
- net Net-(BT1-+): track 0.00 -> 4.08 mm
- net /V_BATT: track 0.00 -> 3.70 mm, vias 0 -> 1
- net Net-(U1-STAT): track 0.00 -> 2.92 mm
- net Net-(U2-SW): track 0.00 -> 2.89 mm
- net Net-(U2-EN): track 0.00 -> 1.97 mm
Other:
- board size 81 x 113 mm -> 166.8 x 113 mm
- board text added: "AA"

Commit message: Update ESP from S3 to WROVER
Changed ESP to be compatible to odroid-go
Parts:
- removed D2: LED, LED_SMD:LED_0603_1608Metric
- removed J2, J3: Conn_01x02_Female, Connector_JST:JST_PH_B2B-PH-K_1x02_P2.00mm_Vertical
- removed SW6: SW_Push, TheBrutzlers_Lib:RubberpadButton_250µ_250µ
- removed U5: MAX98357AETE+T, Package_DFN_QFN:QFN-16-1EP_3x3mm_P0.5mm_EP1.45x1.45mm
- removed U6: 02FVS3, TheBrutzlers_Lib:02FVS3
- added C10: 100n, Capacitor_SMD:C_1206_3216Metric, F.Cu at (247.4, 76.8)
- added C11: 4µ7, Capacitor_SMD:C_1206_3216Metric, F.Cu at (247.4, 80.2)
- added C12: 100n, Capacitor_SMD:C_1206_3216Metric, F.Cu at (262.4, 70.1)
- added C13: 100n, Capacitor_SMD:C_1206_3216Metric, F.Cu at (262.4, 73.5)
- added C14: 4µ7, Capacitor_SMD:C_1206_3216Metric, F.Cu at (262.4, 76.8)
- added C15: 220p, Capacitor_SMD:C_0603_1608Metric, F.Cu at (267.3, 69.7)
- added C16: 220p, Capacitor_SMD:C_0603_1608Metric, F.Cu at (267.3, 72.2)
- added C17: 4µ7, Capacitor_SMD:C_1206_3216Metric, F.Cu at (262.4, 80.2)
- added CN1: PJ-3043-B, easyeda2kicad:AUDIO-TH_PJ-3043-B, F.Cu at (193.6, 144.4)
- added FB3: FerriteBead_Small, Inductor_SMD:L_0805_2012Metric, F.Cu at (271.6, 69.8)
- added FB4: FerriteBead_Small, Inductor_SMD:L_0805_2012Metric, F.Cu at (271.6, 72.6)
- added FB5: FerriteBead_Small, Inductor_SMD:L_0805_2012Metric, F.Cu at (271.6, 75.3)
- added H1: MountingHole, MountingHole:MountingHole_2.2mm_M2, F.Cu at (194.5, 151.8)
- added H2: MountingHole, MountingHole:MountingHole_2.2mm_M2, F.Cu at (194.5, 135.8)
- added J10: Conn_01x01_Pin, TheBrutzlers_Lib:NINTENDO_MINUS, F.Cu at (138.5, 104.3)
- added J6: Conn_01x05_Pin, Connector_PinHeader_2.00mm:PinHeader_1x05_P2.00mm_Vertical, F.Cu at (185.8, 110.0)
- added J7: Conn_01x18_Socket, TheBrutzlers_Lib:solder connector 0.8mm 18 pin, F.Cu at (251.0, 89.4)
- added J8: Conn_01x05_Socket, Connector_PinHeader_2.00mm:PinHeader_1x05_P2.00mm_Vertical, F.Cu at (122.0, 104.3)
- added J9: Conn_01x01_Pin, TheBrutzlers_Lib:NINTENDO_PLUS, F.Cu at (182.1, 104.3)
- added Q2: BC817, Package_TO_SOT_SMD:SOT-23, F.Cu at (247.0, 88.9)
- added Q3: BC817, Package_TO_SOT_SMD:SOT-23, F.Cu at (272.1, 83.4)
- added Q4: BC817, Package_TO_SOT_SMD:SOT-23, F.Cu at (247.0, 93.5)
- added R24: 22, Resistor_SMD:R_0603_1608Metric_Pad0.98x0.95mm_HandSolder, F.Cu at (233.7, 77.2)
- added R33: 22, Resistor_SMD:R_0603_1608Metric_Pad0.98x0.95mm_HandSolder, F.Cu at (238.1, 74.7)
- added R34: 22, Resistor_SMD:R_0603_1608Metric_Pad0.98x0.95mm_HandSolder, F.Cu at (238.1, 77.2)
- added R35: 22, Resistor_SMD:R_0603_1608Metric_Pad0.98x0.95mm_HandSolder, F.Cu at (238.1, 79.7)
- added R36: 22, Resistor_SMD:R_0603_1608Metric_Pad0.98x0.95mm_HandSolder, F.Cu at (238.1, 82.3)
- added R37: 5K1, Resistor_SMD:R_0603_1608Metric_Pad0.98x0.95mm_HandSolder, F.Cu at (238.1, 84.8)
- added R38: 5K1, Resistor_SMD:R_0603_1608Metric_Pad0.98x0.95mm_HandSolder, F.Cu at (238.1, 87.3)
- added R39: 5K1, Resistor_SMD:R_0603_1608Metric_Pad0.98x0.95mm_HandSolder, F.Cu at (238.1, 89.8)
- added R40: 5K1, Resistor_SMD:R_0603_1608Metric_Pad0.98x0.95mm_HandSolder, F.Cu at (242.4, 69.7)
- added R41: 5K1, Resistor_SMD:R_0603_1608Metric_Pad0.98x0.95mm_HandSolder, F.Cu at (242.4, 72.2)
- added R42: 5K1, Resistor_SMD:R_0603_1608Metric_Pad0.98x0.95mm_HandSolder, F.Cu at (242.4, 74.7)
- added R43: 22, Resistor_SMD:R_0603_1608Metric_Pad0.98x0.95mm_HandSolder, F.Cu at (242.4, 77.2)
- added R44: 22, Resistor_SMD:R_0603_1608Metric_Pad0.98x0.95mm_HandSolder, F.Cu at (242.4, 79.7)
- added U10: CH340K, TheBrutzlers_Lib:SSOP-10_3.9x4.9mm_P1.00mm_EP_3mmx2mm, F.Cu at (134.8, 50.8)
- added U11: ESP32-WROVER-E-N8R8, easyeda2kicad:WIFI-SMD_ESP32-WROVER-IE8MB, F.Cu at (181.2, 69.8)
- BT1, BT2, R6, R7, SW1, SW8: moved to F.Cu
- J4, J7, LS1, U8: moved to B.Cu
- Q1: value BC807 -> BC817
- R10, R32, R8: footprint Resistor_SMD:R_0603_1608Metric_Pad0.98x0.95mm_HandSolder -> Resistor_SMD:R_0603_1608Metric
- R11, R14: value 5K1 -> 100K
- R23: value 10 -> 100K
- R26: value 10 -> 4R7
- U1: value MCP73831-2-OT -> HE6250xx; footprint Package_TO_SOT_SMD:SOT-23-5 -> Package_TO_SOT_SMD:SOT-89-3
- U3: value ESP32-S3-WROOM-2 -> PAM8406D; footprint RF_Module:ESP32-S3-WROOM-2 -> Package_SO:SOP-16_3.9x9.9mm_P1.27mm
- U4: value 3_2_ZOLL_ILI9341 -> MAX98357AETE+T; footprint TheBrutzlers_Lib:ILI9341_3_2_ZOLL -> Package_DFN_QFN:QFN-16-1EP_3x3mm_P0.5mm_EP1.45x1.45mm
- moved U4 236.5 mm to (241.4, 93.7)
- moved J1 150.3 mm to (122.8, 51.8), turned to -90 degrees
- moved U7 148.4 mm to (123.5, 72.6), turned to 90 degrees
- moved SW7 144.4 mm to (178.4, 90.2)
- moved R11 135.7 mm to (267.4, 82.3), turned to 0 degrees
- moved R32 131.3 mm to (267.3, 79.7), turned to 0 degrees
- moved SW13 126.2 mm to (233.0, 93.1)
- moved LS1 122.3 mm to (178.1, 142.4), turned to 90 degrees
- moved R19 110.4 mm to (233.7, 72.2), turned to 0 degrees
- moved R23 108.0 mm to (233.7, 74.7), turned to 0 degrees
- moved R18 107.9 mm to (233.7, 69.7), turned to 0 degrees
- moved Q1 106.8 mm to (247.0, 84.2), turned to 0 degrees
- moved R14 104.6 mm to (267.4, 84.8)
- moved R17 102.9 mm to (229.4, 89.8), turned to 0 degrees
- moved R31 101.9 mm to (238.1, 72.2), turned to 0 degrees
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Connections:
- C6 pad 1: Net-(C6-Pad1) -> /SPK+
- C7 pad 2: Net-(C7-Pad2) -> /SPK-
- FB1 pad 1: Net-(U5-OUTN) -> Net-(U4-OUTN)
- FB1 pad 2: Net-(C7-Pad2) -> /SPK-
- FB2 pad 1: Net-(U5-OUTP) -> Net-(U4-OUTP)
- FB2 pad 2: Net-(C6-Pad1) -> /SPK+
- J4 pad 10: Net-(J4-Pin_10) -> +3V3
- LS1 pad 1: Net-(C7-Pad2) -> /FRONT_BUTTONS/SPK-
- LS1 pad 2: Net-(C6-Pad1) -> /FRONT_BUTTONS/SPK+
- Q1 pad 2: +3V3 -> /RTS
- Q1 pad 3: Net-(J4-Pin_10) -> /EN
- R10 pad 1: Net-(U1-STAT) -> Net-(U4-GAIN_SLOT)
- R10 pad 2: Net-(D2-K) -> GND
- R11 pad 1: Net-(U3-EN) -> Net-(C12-Pad2)
- R11 pad 2: +3V3 -> Net-(U3-INL)
- R14 pad 1: /KEY_VOL_BOOT -> Net-(C13-Pad2)
- R14 pad 2: +3V3 -> Net-(U3-INR)
- R15 pad 1: GND -> Net-(U10-V3)
- R15 pad 2: Net-(U3-IO46) -> +3V3
- R20 pad 1: +3V3 -> /I2S_EN
- R20 pad 2: Net-(U5-GAIN_SLOT) -> +3V3
- R21 pad 1: Net-(U5-GAIN_SLOT) -> Net-(U3-PVDDL)
- R21 pad 2: GND -> Net-(U3-MODE)
- R22 pad 1: Net-(U5-SD_MODE) -> Net-(U3-MODE)
- R22 pad 2: +3V3 -> Net-(J6-Pin_1)
- R23 pad 1: GND -> /LCD_BCKL
- R23 pad 2: Net-(J6-Pin_7) -> GND
- R25 pad 1: Net-(Q1-B) -> /DTR
- R25 pad 2: /LCD_BCKL -> Net-(Q1-B)
- R26 pad 1: GND -> Net-(Q2-C)
- R31 pad 1: Net-(U3-IO14) -> /RTS
- R31 pad 2: /LCD_~{CS} -> Net-(Q4-B)
- R32 pad 1: GND -> Net-(U3-PVDDL)
- R32 pad 2: /LCD_~{CS} -> Net-(Q3-C)
- R8 pad 1: Net-(U1-PROG) -> +3V3
- R8 pad 2: GND -> Net-(U4-GAIN_SLOT)
- U1 pad 1: Net-(U1-STAT) -> GND
- U1 pad 2: GND -> /VUSB
- U3 pad 1: GND -> Net-(U3-+OUT_L)
- U3 pad 10: /KEY_START -> Net-(U3-INR)
- U3 pad 11: /KEY_MENU -> Net-(J6-Pin_1)
- U3 pad 12: /KEY_OPTION -> Net-(Q3-C)
- U3 pad 13: /D+ -> Net-(U3-PVDDL)
- U3 pad 14: /D- -> Net-(J6-Pin_1)
- U3 pad 15: /LCD_RESET -> Net-(J6-Pin_1)
- U3 pad 16: Net-(U3-IO46) -> Net-(U3-+OUT_R)
- U3 pad 2: +3V3 -> Net-(J6-Pin_1)
- U3 pad 3: Net-(U3-EN) -> Net-(J6-Pin_1)
- U3 pad 4: /V_BAT_ADC -> Net-(U3-PVDDL)
- U3 pad 5: /KEY_B -> Net-(U3-PVDDL)
- U3 pad 6: /KEY_UP -> Net-(U3-PVDDL)
- U3 pad 7: /KEY_LEFT -> Net-(U3-INL)
- U3 pad 8: /KEY_A -> Net-(U3-VREF)
- U3 pad 9: /KEY_SELECT -> Net-(U3-MODE)
- U4 pad 1: +3V3 -> /I2S_DATA
- U4 pad 10: unconnected-(U4-T_SCK-Pad10) -> Net-(U4-OUTN)
- U4 pad 11: unconnected-(U4-T_CS-Pad11) -> GND
- U4 pad 12: unconnected-(U4-T_MOSI-Pad12) -> (no net)
- U4 pad 13: unconnected-(U4-T_MISO-Pad13) -> (no net)
- U4 pad 14: unconnected-(U4-T_IRQ-Pad14) -> /I2S_WS
- U4 pad 15: /SD_CLK -> GND
- U4 pad 16: /SD_MISO -> /I2S_BCK
- U4 pad 17: /SD_MOSI -> GND
- U4 pad 2: GND -> Net-(U4-GAIN_SLOT)
- U4 pad 3: /LCD_~{CS} -> GND
- U4 pad 4: /LCD_RESET -> /I2S_EN
- U4 pad 5: /LCD_DC -> (no net)
- U4 pad 6: /LCD_MOSI -> (no net)
- U4 pad 7: /LCD_CLK -> +3V3
- U4 pad 8: Net-(J4-Pin_10) -> +3V3
- U4 pad 9: unconnected-(U4-MISO-Pad9) -> Net-(U4-OUTP)
- U7 pad A: /KEY_OPTION -> /KEY_MENU
- U7 pad S: /KEY_MENU -> /KEY_OPTION
- U8 pad 1: /FRONT_BUTTONS/FRONT_SD_MISO -> /SPK-
- U8 pad 10: /FRONT_BUTTONS/FRONT_GND -> GND
- U8 pad 11: /FRONT_BUTTONS/KEY_DOWN -> /KEY_DOWN
- U8 pad 12: /FRONT_BUTTONS/KEY_B -> /KEY_B
- U8 pad 13: /FRONT_BUTTONS/KEY_UP -> /KEY_UP
- U8 pad 14: /FRONT_BUTTONS/KEY_A -> /KEY_A
- U8 pad 15: /FRONT_BUTTONS/KEY_LEFT -> /KEY_LEFT
- U8 pad 16: /FRONT_BUTTONS/KEY_SELECT -> /KEY_SELECT
- U8 pad 17: /FRONT_BUTTONS/KEY_RIGHT -> /KEY_RIGHT
- U8 pad 18: /FRONT_BUTTONS/KEY_START -> /KEY_START
- U8 pad 19: /FRONT_BUTTONS/FRONT_3V3 -> +3V3
- U8 pad 2: /FRONT_BUTTONS/FRONT_GND -> /SPK+
- U8 pad 20: /FRONT_BUTTONS/FRONT_GND -> GND
- U8 pad 3: /FRONT_BUTTONS/FRONT_SD_CLK -> GND
- U8 pad 4: /FRONT_BUTTONS/FRONT_GND -> GND
- U8 pad 5: /FRONT_BUTTONS/FRONT_SD_MOSI -> /SD_MOSI
- U8 pad 6: /FRONT_BUTTONS/FRONT_GND -> /SD_MISO
- U8 pad 7: /FRONT_BUTTONS/FRONT_SD_CS -> /SD_CS
- U8 pad 8: /FRONT_BUTTONS/FRONT_GND -> /SD_CLK
- U8 pad 9: /FRONT_BUTTONS/FRONT_GND -> GND
- U9 pad 14: /FRONT_BUTTONS/GND -> /FRONT_BUTTONS/SD_CLK
- U9 pad 16: /FRONT_BUTTONS/GND -> /FRONT_BUTTONS/SD_MISO
- U9 pad 17: /FRONT_BUTTONS/SD_CLK -> /FRONT_BUTTONS/GND
- U9 pad 19: /FRONT_BUTTONS/SD_MISO -> /FRONT_BUTTONS/SPK-
- U9 pad 20: /FRONT_BUTTONS/GND -> /FRONT_BUTTONS/SPK+
Routing:
- net /VUSB: track 4.19 -> 15.0 mm
- net GND: track 21.8 -> 14.3 mm
- net Net-(U1-PROG): track 4.21 -> 0.00 mm
- net Net-(U1-STAT): track 2.92 -> 0.00 mm
- net Net-(BT1-+): track 4.08 -> 4.70 mm
- net (no net): vias 0 -> 23
Other:
- board size 166.8 x 113 mm -> 99.4 x 130.1 mm
