File: ILI9341_ESP32/AUDIO.kicad_sch (KiCad schematic)
At the start: 3 parts, among them CN1 PJ-3043-B, J2 Conn_01x04_Pin, J3 Conn_01x04_Socket

Commit message: update nimh charger and battery protection
Parts:
- CN1: LCSC (none) -> C2682182; LCSC Part C2682182 -> (none)
Changed lines of the file:
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@@
 			)
 		)
-		(property "LCSC Part" "C2682182"
+		(property "LCSC Part" ""
 			(at 199.39 101.6 0)
 			(effects
@@
 			(at 199.39 81.28 0)
 			(effects
+				(font
+					(size 1.27 1.27)
+				)
+				(hide yes)
+			)
+		)
+		(property "LCSC" "C2682182"
+			(at 199.39 81.28 0)
+			(effects

Commit message: ordered Version
Parts:
- CN1: SOURCED jop -> (none)
Changed lines of the file:
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@@
 			)
 		)
-		(property "SOURCED" "jop"
+		(property "SOURCED" ""
 			(at 199.39 81.28 0)
 			(effects
