File: ILI9341_ESP32/untitled.kicad_sch (KiCad schematic)
At the start: 16 parts, among them J7 Conn_01x32, Q5 Q_PMOS_GSD, Q6 BC817, U5 MCP23017_SO, U6 MCP23017_SO

Commit message: Update PCB and add RGB
Parts:
- C21, C22: footprint Capacitor_SMD:C_1206_3216Metric -> Capacitor_SMD:C_0603_1608Metric; LCSC C464972 -> (none)
Changed lines of the file:
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@@
 			)
 		)
-		(property "Footprint" "Capacitor_SMD:C_1206_3216Metric"
+		(property "Footprint" "Capacitor_SMD:C_0603_1608Metric"
 			(at 62.5348 66.04 0)
 			(effects
@@
 			)
 		)
-		(property "LCSC" "C464972"
+		(property "LCSC" ""
 			(at 63.5 69.85 0)
 			(effects
@@
 			)
 		)
-		(property "Footprint" "Capacitor_SMD:C_1206_3216Metric"
+		(property "Footprint" "Capacitor_SMD:C_0603_1608Metric"
 			(at 75.2348 119.38 0)
 			(effects
@@
 			)
 		)
-		(property "LCSC" "C464972"
+		(property "LCSC" ""
 			(at 76.2 123.19 0)
 			(effects

Commit message: ordered Version
Parts:
- C21, C22, C23, C24, C25, D5, J7, Q6, R24, R29, R30, R33, R34, U5, U6: SOURCED jop -> (none)
- Q5: value Q_PMOS_GSD -> PMOS; SOURCED jop -> (none)
Connections:
- net CHARGER_EN: now reaches U6.28 (GPA7)
Changed lines of the file:
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@@
 	(wire
 		(pts
+			(xy 29.845 156.21) (xy 144.145 156.21)
+		)
+		(stroke
+			(width 0)
+			(type default)
+		)
+	)
+	(wire
+		(pts
 			(xy 193.04 111.76) (xy 205.74 111.76)
 		)
@@
 	(wire
 		(pts
+			(xy 144.145 137.16) (xy 144.145 156.21)
+		)
+		(stroke
+			(width 0)
+			(type default)
+		)
+	)
+	(wire
+		(pts
 			(xy 76.2 119.38) (xy 104.14 119.38)
 		)
@@
 	(wire
 		(pts
+			(xy 139.7 137.16) (xy 144.145 137.16)
+		)
+		(stroke
+			(width 0)
+			(type default)
+		)
+	)
+	(wire
+		(pts
 			(xy 139.7 119.38) (xy 154.94 119.38)
 		)
@@
 		)
 	)
+	(hierarchical_label "CHARGER_EN"
+		(shape output)
+		(at 29.845 156.21 180)
+		(fields_autoplaced yes)
+		(effects
+			(font
+				(size 1.27 1.27)
+			)
+			(justify right)
+		)
+	)
 	(hierarchical_label "CARD_SDA"
 		(shape bidirectional)
@@
 			)
 		)
-		(property "SOURCED" "jop"
+		(property "SOURCED" ""
 			(at 78.105 24.765 0)
 			(effects
@@
 			)
 		)
-		(property "SOURCED" "jop"
+		(property "SOURCED" ""
 			(at 148.59 134.62 0)
 			(effects
@@
 			)
 		)
-		(property "SOURCED" "jop"
+		(property "SOURCED" ""
 			(at 66.04 119.38 0)
 			(effects
@@
 			)
 		)
-		(property "SOURCED" "jop"
+		(property "SOURCED" ""
 			(at 121.92 116.84 0)
 			(effects
@@
 			)
 		)
-		(property "SOURCED" "jop"
+		(property "SOURCED" ""
 			(at 210.82 86.36 0)
 			(effects
@@
 			)
 		)
-		(property "SOURCED" "jop"
+		(property "SOURCED" ""
 			(at 125.095 31.75 0)
 			(effects
@@
 			)
 		)
-		(property "SOURCED" "jop"
+		(property "SOURCED" ""
 			(at 183.515 52.07 0)
 			(effects
@@
 			)
 		)
-		(property "Value" "Q_PMOS_GSD"
+		(property "Value" "PMOS"
 			(at 85.725 28.575 90)
 			(effects
@@
 			)
 		)
-		(property "SOURCED" "jop"
+		(property "SOURCED" ""
 			(at 76.835 34.29 0)
 			(effects
@@
 			)
 		)
-		(property "SOURCED" "jop"
+		(property "SOURCED" ""
 			(at 99.06 63.5 0)
 			(effects
@@
 			)
 		)
-		(property "SOURCED" "jop"
+		(property "SOURCED" ""
 			(at 63.5 69.85 0)
 			(effects
@@
 			)
 		)
-		(property "SOURCED" "jop"
+		(property "SOURCED" ""
 			(at 53.34 66.04 0)
 			(effects
@@
 			)
 		)
-		(property "SOURCED" "jop"
+		(property "SOURCED" ""
 			(at 160.655 134.62 0)
 			(effects
@@
 			)
 		)
-		(property "SOURCED" "jop"
+		(property "SOURCED" ""
 			(at 156.21 139.7 0)
 			(effects
@@
 			)
 		)
-		(property "SOURCED" "jop"
+		(property "SOURCED" ""
 			(at 71.12 39.37 0)
 			(effects
@@
 			)
 		)
-		(property "SOURCED" "jop"
+		(property "SOURCED" ""
 			(at 140.97 90.17 0)
 			(effects
@@
 			)
 		)
-		(property "SOURCED" "jop"
+		(property "SOURCED" ""
 			(at 76.2 123.19 0)
 			(effects
